File: MoteinoM0CAM-M8.brd (EAGLE design)
At the start: 22.6 x 22.2 mm, 17 parts

Commit message: moved 4.7uF
Parts:
- removed C3: 4.7uF, SparkFun-Capacitors:0603
- added C4: 4.7uF, SparkFun-Capacitors:0603
Connections:
- net GND: now also C4.2; no longer C3.2
- net VCC: now also C4.1
- net VIN: no longer C3.1
Routing:
- net VCC: track 18.8 -> 22.2 mm
- net VIN: track 10.7 -> 7.70 mm
- net GND: vias 22 -> 11
Changed lines of the file:
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@@
 <attribute name="VALUE" x="8.001" y="2.286" size="0.6096" layer="27" font="vector" ratio="20" align="top-center"/>
 </element>
-<element name="C3" library="SparkFun-Capacitors" library_urn="urn:adsk.eagle:library:510" package="0603" package3d_urn="urn:adsk.eagle:package:37414/1" value="4.7uF" x="12.319" y="0" smashed="yes" rot="R180">
-<attribute name="NAME" x="12.319" y="-0.762" size="0.6096" layer="25" font="vector" ratio="20" rot="R180" align="bottom-center"/>
-<attribute name="PROD_ID" value="CAP-08280" x="12.319" y="0" size="1.778" layer="27" rot="R180" display="off"/>
-<attribute name="VALUE" x="12.319" y="0.762" size="0.6096" layer="27" font="vector" ratio="20" rot="R180" align="top-center"/>
+<element name="C4" library="SparkFun-Capacitors" library_urn="urn:adsk.eagle:library:510" package="0603" package3d_urn="urn:adsk.eagle:package:37414/1" value="4.7uF" x="12.319" y="0.127" smashed="yes" rot="R180">
+<attribute name="NAME" x="12.319" y="-0.635" size="0.6096" layer="25" font="vector" ratio="20" rot="R180" align="bottom-center"/>
+<attribute name="PROD_ID" value="CAP-08280" x="12.319" y="0.127" size="1.778" layer="27" rot="R180" display="off"/>
+<attribute name="VALUE" x="12.319" y="0.889" size="0.6096" layer="27" font="vector" ratio="20" rot="R180" align="top-center"/>
 </element>
 </elements>
@@
 <contactref element="C2" pad="2"/>
 <contactref element="U$18" pad="1"/>
-<contactref element="C3" pad="2"/>
-<wire x1="2.4384" y1="3.048" x2="1.4224" y2="3.048" width="0.1524" layer="1"/>
-<wire x1="1.4224" y1="3.048" x2="1.27" y2="2.921" width="0.1524" layer="1"/>
-<wire x1="2.4384" y1="3.048" x2="2.539996875" y2="2.87019375" width="0.1524" layer="1"/>
-<wire x1="21.5392" y1="3.048" x2="1.4224" y2="3.048" width="0.1524" layer="16"/>
-<wire x1="1.4224" y1="3.048" x2="1.27" y2="2.921" width="0.1524" layer="16"/>
-<wire x1="21.5392" y1="3.048" x2="21.59" y2="2.921" width="0.1524" layer="16"/>
 <polygon width="0.1524" layer="16" isolate="0.3048">
 <vertex x="0.127" y="20.447"/>
@@
 <vertex x="0.127" y="-1.143"/>
 </polygon>
-<via x="3.429" y="9.271" extent="1-16" drill="0.35"/>
+<contactref element="C4" pad="2"/>
+<wire x1="2.4384" y1="3.048" x2="1.4224" y2="3.048" width="0.1524" layer="1"/>
+<wire x1="1.4224" y1="3.048" x2="1.27" y2="2.921" width="0.1524" layer="1"/>
+<wire x1="2.4384" y1="3.048" x2="2.539996875" y2="2.87019375" width="0.1524" layer="1"/>
+<wire x1="21.5392" y1="3.048" x2="1.4224" y2="3.048" width="0.1524" layer="16"/>
+<wire x1="1.4224" y1="3.048" x2="1.27" y2="2.921" width="0.1524" layer="16"/>
+<wire x1="21.5392" y1="3.048" x2="21.59" y2="2.921" width="0.1524" layer="16"/>
+<via x="10.668" y="13.97" extent="1-16" drill="0.35"/>
+<via x="13.589" y="14.224" extent="1-16" drill="0.35"/>
+<via x="11.557" y="10.795" extent="1-16" drill="0.35"/>
+<via x="18.669" y="16.129" extent="1-16" drill="0.35"/>
+<via x="19.177" y="10.033" extent="1-16" drill="0.35"/>
+<via x="9.271" y="0.381" extent="1-16" drill="0.35"/>
+<via x="5.461" y="3.937" extent="1-16" drill="0.35"/>
 <via x="4.826" y="6.858" extent="1-16" drill="0.35"/>
-<via x="5.588" y="3.937" extent="1-16" drill="0.35"/>
-<via x="5.588" y="1.905" extent="1-16" drill="0.35"/>
-<via x="3.048" y="1.905" extent="1-16" drill="0.35"/>
-<via x="9.144" y="1.27" extent="1-16" drill="0.35"/>
-<via x="9.144" y="-0.635" extent="1-16" drill="0.35"/>
-<via x="10.922" y="1.397" extent="1-16" drill="0.35"/>
-<via x="13.462" y="1.524" extent="1-16" drill="0.35"/>
-<via x="19.431" y="0" extent="1-16" drill="0.35"/>
-<via x="19.05" y="6.858" extent="1-16" drill="0.35"/>
-<via x="19.05" y="9.398" extent="1-16" drill="0.35"/>
-<via x="18.923" y="11.43" extent="1-16" drill="0.35"/>
-<via x="18.923" y="13.462" extent="1-16" drill="0.35"/>
-<via x="3.048" y="11.811" extent="1-16" drill="0.35"/>
-<via x="3.175" y="4.064" extent="1-16" drill="0.35"/>
-<via x="3.048" y="19.177" extent="1-16" drill="0.35"/>
-<via x="4.953" y="19.304" extent="1-16" drill="0.35"/>
-<via x="17.78" y="19.177" extent="1-16" drill="0.35"/>
-<via x="18.923" y="17.526" extent="1-16" drill="0.35"/>
-<via x="17.653" y="16.383" extent="1-16" drill="0.35"/>
-<via x="18.923" y="15.494" extent="1-16" drill="0.35"/>
-<wire x1="17.653" y1="16.383" x2="18.923" y2="15.494" width="0" layer="19" extent="1-1"/>
+<via x="3.302" y="9.906" extent="1-16" drill="0.35"/>
+<via x="3.302" y="14.986" extent="1-16" drill="0.35"/>
+<via x="4.445" y="19.304" extent="1-16" drill="0.35"/>
 </signal>
 <signal name="SDA">
@@
 <contactref element="LDO" pad="1"/>
 <contactref element="C1" pad="1"/>
-<contactref element="C3" pad="1"/>
-<wire x1="16.168" y1="0" x2="13.169" y2="0" width="0.1524" layer="1"/>
+<wire x1="16.256" y1="1.2192" x2="16.256" y2="0" width="0.1524" layer="1"/>
+<wire x1="16.8656" y1="1.8288" x2="16.256" y2="1.2192" width="0.1524" layer="1"/>
+<wire x1="17.4752" y1="1.8288" x2="16.8656" y2="1.8288" width="0.1524" layer="1"/>
+<wire x1="17.6784" y1="2.032" x2="17.4752" y2="1.8288" width="0.1524" layer="1"/>
+<wire x1="18.0848" y1="2.032" x2="17.6784" y2="2.032" width="0.1524" layer="1"/>
+<wire x1="16.256" y1="0" x2="16.168" y2="0" width="0.1524" layer="1"/>
+<wire x1="18.0848" y1="2.032" x2="18.1911" y2="2.098" width="0.1524" layer="1"/>
 <wire x1="18.8976" y1="2.032" x2="18.288" y2="2.032" width="0.1524" layer="1"/>
 <wire x1="19.1008" y1="1.8288" x2="18.8976" y2="2.032" width="0.1524" layer="1"/>
@@
 <wire x1="18.288" y1="2.032" x2="18.1911" y2="2.098" width="0.1524" layer="1"/>
 <wire x1="21.5392" y1="0.4064" x2="21.59" y2="0.381" width="0.1524" layer="1"/>
-<wire x1="16.256" y1="1.2192" x2="16.256" y2="0" width="0.1524" layer="1"/>
-<wire x1="16.8656" y1="1.8288" x2="16.256" y2="1.2192" width="0.1524" layer="1"/>
-<wire x1="17.4752" y1="1.8288" x2="16.8656" y2="1.8288" width="0.1524" layer="1"/>
-<wire x1="17.6784" y1="2.032" x2="17.4752" y2="1.8288" width="0.1524" layer="1"/>
-<wire x1="18.0848" y1="2.032" x2="17.6784" y2="2.032" width="0.1524" layer="1"/>
-<wire x1="16.256" y1="0" x2="16.168" y2="0" width="0.1524" layer="1"/>
-<wire x1="18.0848" y1="2.032" x2="18.1911" y2="2.098" width="0.1524" layer="1"/>
 <wire x1="21.59" y1="0.381" x2="22.86" y2="0.381" width="0" layer="19" extent="1-1"/>
 </signal>
@@
 <contactref element="C2" pad="1"/>
 <contactref element="LDO" pad="5"/>
-<wire x1="13.8176" y1="3.048" x2="13.208" y2="3.048" width="0.1524" layer="1"/>
-<wire x1="14.8336" y1="2.032" x2="13.8176" y2="3.048" width="0.1524" layer="1"/>
-<wire x1="15.4432" y1="2.032" x2="14.8336" y2="2.032" width="0.1524" layer="1"/>
+<contactref element="C4" pad="1"/>
+<wire x1="13.208" y1="3.048" x2="13.208" y2="0.2032" width="0.1524" layer="1"/>
+<wire x1="15.4432" y1="1.8288" x2="15.4432" y2="2.032" width="0.1524" layer="1"/>
+<wire x1="13.8176" y1="0.2032" x2="15.4432" y2="1.8288" width="0.1524" layer="1"/>
+<wire x1="13.208" y1="0.2032" x2="13.8176" y2="0.2032" width="0.1524" layer="1"/>
 <wire x1="15.4432" y1="2.032" x2="15.5909" y2="2.098" width="0.1524" layer="1"/>
+<wire x1="13.208" y1="0.2032" x2="13.169" y2="0.127" width="0.1524" layer="1"/>
 <wire x1="15.6464" y1="6.096" x2="15.6464" y2="6.9088" width="0.1524" layer="1"/>
 <wire x1="14.224" y1="4.6736" x2="15.6464" y2="6.096" width="0.1524" layer="1"/>
@@
 <wire x1="7.112" y1="0" x2="7.088" y2="0" width="0.1524" layer="1"/>
 </signal>
+<signal name="N$13">
+<via x="18.542" y="18.796" extent="1-16" drill="0.35"/>
+</signal>
 </signals>

Commit message: final
Parts:
- renumbered C4 to C3
Changed lines of the file:
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@@
 <attribute name="VALUE" x="8.001" y="2.286" size="0.6096" layer="27" font="vector" ratio="20" align="top-center"/>
 </element>
-<element name="C4" library="SparkFun-Capacitors" library_urn="urn:adsk.eagle:library:510" package="0603" package3d_urn="urn:adsk.eagle:package:37414/1" value="4.7uF" x="12.319" y="0.127" smashed="yes" rot="R180">
+<element name="C3" library="SparkFun-Capacitors" library_urn="urn:adsk.eagle:library:510" package="0603" package3d_urn="urn:adsk.eagle:package:37414/1" value="4.7uF" x="12.319" y="0.127" smashed="yes" rot="R180">
 <attribute name="NAME" x="12.319" y="-0.635" size="0.6096" layer="25" font="vector" ratio="20" rot="R180" align="bottom-center"/>
 <attribute name="PROD_ID" value="CAP-08280" x="12.319" y="0.127" size="1.778" layer="27" rot="R180" display="off"/>
@@
 <vertex x="0.127" y="-1.143"/>
 </polygon>
-<contactref element="C4" pad="2"/>
+<contactref element="C3" pad="2"/>
 <wire x1="2.4384" y1="3.048" x2="1.4224" y2="3.048" width="0.1524" layer="1"/>
 <wire x1="1.4224" y1="3.048" x2="1.27" y2="2.921" width="0.1524" layer="1"/>
@@
 <contactref element="C2" pad="1"/>
 <contactref element="LDO" pad="5"/>
-<contactref element="C4" pad="1"/>
+<contactref element="C3" pad="1"/>
 <wire x1="13.208" y1="3.048" x2="13.208" y2="0.2032" width="0.1524" layer="1"/>
 <wire x1="15.4432" y1="1.8288" x2="15.4432" y2="2.032" width="0.1524" layer="1"/>
